File: Pinecil_LEDring.kicad_sch (KiCad schematic)
At the start: 7 parts

Commit message: Add files via upload
Parts:
- removed D3: LED, LED_SMD:LED_0603_1608Metric_Pad1.05x0.95mm_HandSolder, symbol Device:LED
- removed D5: LED, LED_SMD:LED_1206_3216Metric_Pad1.42x1.75mm_HandSolder, symbol Device:LED
- added R3: R_Small, Resistors_SMD:R_0603_HandSoldering, symbol Device:R_Small
Connections:
- net +5V: now also R3.1
- net GND: now also D4.1 (K)
- net at D4.2 (A): now also R3.2
Other:
- moved on the sheet: D4
Changed lines of the file:
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@@
 (kicad_sch (version 20211123) (generator eeschema)
   (paper "A4")
+  (junction (at 72.39 67.31) (diameter 0) (color 0 0 0 0)
+  )
   (junction (at 72.39 63.5) (diameter 0) (color 0 0 0 0)
   )
   (junction (at 96.52 64.77) (diameter 0) (color 0 0 0 0)
   )
+  (junction (at 96.52 67.31) (diameter 0) (color 0 0 0 0)
+  )
   (wire (pts (xy 80.01 60.96) (xy 81.28 60.96))
+    (stroke (width 0) (type default) (color 0 0 0 0))
+  )
+  (wire (pts (xy 72.39 72.39) (xy 72.39 67.31))
     (stroke (width 0) (type default) (color 0 0 0 0))
   )
@@
     (stroke (width 0) (type default) (color 0 0 0 0))
   )
+  (wire (pts (xy 96.52 72.39) (xy 96.52 67.31))
+    (stroke (width 0) (type default) (color 0 0 0 0))
+  )
+  (wire (pts (xy 80.01 72.39) (xy 81.28 72.39))
+    (stroke (width 0) (type default) (color 0 0 0 0))
+  )
   (wire (pts (xy 96.52 67.31) (xy 88.9 67.31))
+    (stroke (width 0) (type default) (color 0 0 0 0))
+  )
+  (wire (pts (xy 74.93 72.39) (xy 72.39 72.39))
     (stroke (width 0) (type default) (color 0 0 0 0))
   )
@@
     (stroke (width 0) (type default) (color 0 0 0 0))
   )
+  (wire (pts (xy 88.9 72.39) (xy 96.52 72.39))
+    (stroke (width 0) (type default) (color 0 0 0 0))
+  )
   (wire (pts (xy 88.9 60.96) (xy 96.52 60.96))
     (stroke (width 0) (type default) (color 0 0 0 0))
@@
     (stroke (width 0) (type default) (color 0 0 0 0))
   )
-  (symbol (lib_id "Device:LED") (at 95.25 78.74 180) (unit 1)
+  (symbol (lib_id "Device:LED") (at 85.09 72.39 180) (unit 1)
     (in_bom yes) (on_board yes) (fields_autoplaced)
-    (property "Reference" "D4" (id 0) (at 96.8375 72.8812 0))
-    (property "Value" "LED" (id 1) (at 96.8375 75.4181 0))
-    (property "Footprint" "LED_SMD:LED_0805_2012Metric_Pad1.15x1.40mm_HandSolder" (id 2) (at 95.25 78.74 0)
+    (property "Reference" "D4" (id 0) (at 86.6775 66.5312 0))
+    (property "Value" "LED" (id 1) (at 86.6775 69.0681 0))
+    (property "Footprint" "LED_SMD:LED_0805_2012Metric_Pad1.15x1.40mm_HandSolder" (id 2) (at 85.09 72.39 0)
       (effects (font (size 1.27 1.27)) hide)
     )
-    (property "Datasheet" "~" (id 3) (at 95.25 78.74 0)
-      (effects (font (size 1.27 1.27)) hide)
-    )
-    (pin "1")
-    (pin "2")
-  )
-  (symbol (lib_id "Device:LED") (at 109.22 78.74 180) (unit 1)
-    (in_bom yes) (on_board yes) (fields_autoplaced)
-    (property "Reference" "D5" (id 0) (at 110.8075 72.8812 0))
-    (property "Value" "LED" (id 1) (at 110.8075 75.4181 0))
-    (property "Footprint" "LED_SMD:LED_1206_3216Metric_Pad1.42x1.75mm_HandSolder" (id 2) (at 109.22 78.74 0)
-      (effects (font (size 1.27 1.27)) hide)
-    )
-    (property "Datasheet" "~" (id 3) (at 109.22 78.74 0)
+    (property "Datasheet" "~" (id 3) (at 85.09 72.39 0)
       (effects (font (size 1.27 1.27)) hide)
     )
@@
     (pin "2")
   )
-  (symbol (lib_id "Device:LED") (at 77.47 78.74 180) (unit 1)
-    (in_bom yes) (on_board yes) (fields_autoplaced)
-    (property "Reference" "D3" (id 0) (at 79.0575 72.8812 0))
-    (property "Value" "LED" (id 1) (at 79.0575 75.4181 0))
-    (property "Footprint" "LED_SMD:LED_0603_1608Metric_Pad1.05x0.95mm_HandSolder" (id 2) (at 77.47 78.74 0)
-      (effects (font (size 1.27 1.27)) hide)
-    )
-    (property "Datasheet" "~" (id 3) (at 77.47 78.74 0)
-      (effects (font (size 1.27 1.27)) hide)
-    )
-    (pin "1")
-    (pin "2")
-  )
   (symbol (lib_id "Device:LED") (at 85.09 60.96 180) (unit 1)
     (in_bom yes) (on_board yes) (fields_autoplaced)
@@
     )
     (property "Datasheet" "~" (id 3) (at 85.09 60.96 0)
+      (effects (font (size 1.27 1.27)) hide)
+    )
+    (pin "1")
+    (pin "2")
+  )
+  (symbol (lib_id "Device:R_Small") (at 77.47 72.39 90) (unit 1)
+    (in_bom yes) (on_board yes) (fields_autoplaced)
+    (property "Reference" "R3" (id 0) (at 77.47 67.9536 90))
+    (property "Value" "R_Small" (id 1) (at 77.47 70.4905 90))
+    (property "Footprint" "Resistors_SMD:R_0603_HandSoldering" (id 2) (at 77.47 72.39 0)
+      (effects (font (size 1.27 1.27)) hide)
+    )
+    (property "Datasheet" "~" (id 3) (at 77.47 72.39 0)
       (effects (font (size 1.27 1.27)) hide)
     )
@@
       (reference "D2") (unit 1) (value "LED") (footprint "LEDs:LED-3MM")
     )
-    (path "/d515bf26-6802-41e5-80f5-3195fb5ae026"
-      (reference "D3") (unit 1) (value "LED") (footprint "LED_SMD:LED_0603_1608Metric_Pad1.05x0.95mm_HandSolder")
-    )
     (path "/1f98925c-dc2a-47a4-a0b2-aac2eba55c9e"
       (reference "D4") (unit 1) (value "LED") (footprint "LED_SMD:LED_0805_2012Metric_Pad1.15x1.40mm_HandSolder")
-    )
-    (path "/530c9832-96ca-43ae-8e01-af845304fd48"
-      (reference "D5") (unit 1) (value "LED") (footprint "LED_SMD:LED_1206_3216Metric_Pad1.42x1.75mm_HandSolder")
     )
     (path "/a16c9c01-f80a-4f76-b742-a3e02c8cdacf"
@@
       (reference "R2") (unit 1) (value "R_Small") (footprint "Resistors_SMD:R_0603_HandSoldering")
     )
+    (path "/fc20b964-3ff2-4571-bb09-91f5d527739f"
+      (reference "R3") (unit 1) (value "R_Small") (footprint "Resistors_SMD:R_0603_HandSoldering")
+    )
   )
