File: Pinecil_LEDring.kicad_pcb (KiCad board)
At the start: 2 copper layers, 21.2 x 17.1 mm, 10 parts

Commit message: Add files via upload
Parts:
- removed the G*** at (146.3, 104.6)
- added D4: LED, LED_SMD:LED_0805_2012Metric_Pad1.15x1.40mm_HandSolder, B.Cu at (146.0, 104.5)
- added R3: R_Small, Resistors_SMD:R_0603_HandSoldering, F.Cu at (139.2, 101.3)
- moved G*** 0.30 mm to (146.0, 104.5)
Routing:
- net +5V: track 1.52 -> 12.1 mm, vias 0 -> 1
- net Net-(D4-Pad2): track 0.00 -> 5.90 mm, vias 0 -> 1
- net GND: track 0.00 -> 4.90 mm, vias 0 -> 1

Commit message: Added updated design files and gerbers
Updated the design off the board to make soldering the wires easier.
Parts:
- removed the G*** at (146.1, 89.3)
- removed the G*** at (146.2, 89.3)
- added G***: LOGO, CustomSilkScreen:BW_herushan_Normal_tinyNB, F.Cu at (146.0, 89.4)
- added G***: LOGO, CustomSilkScreen:BW_herushan_Normal_tinyMask, B.Cu at (146.0, 89.2)
- moved REF** 0.51 mm to (153.0, 93.0)
Routing:
- net GND: track 4.90 -> 33.2 mm, vias 1 -> 3
- net +5V: track 12.1 -> 36.7 mm
Other:
- board text added: "如 山"
